File: analog.kicad_sch (KiCad schematic)
At the start: 20 parts, among them U8 MAX11125

Commit message: remove unneeded components from schema
Parts:
- removed AUDIO1: JACK_TRS_6PINS, audio-jack:CUI_SJ-43516-SMT, symbol jack_trs_6pins_apple:JACK_TRS_6PINS_APPLE
- removed C58, C61: 22uF, Capacitor_SMD:C_0805_2012Metric, symbol Device:C
- removed C59, C62: 220nF, Capacitor_SMD:C_0603_1608Metric, symbol Device:C
- removed L4, L5: 33uH, Inductor_SMD:L_0805_2012Metric_Pad1.15x1.40mm_HandSolder, symbol Device:L_Small
- removed R14, R18, R57: 1.1k, Resistor_SMD:R_0603_1608Metric, symbol Device:R
- removed R15, R19, R58: 549, Resistor_SMD:R_0603_1608Metric, symbol Device:R
- removed R16, R20, R59: 270, Resistor_SMD:R_0603_1608Metric, symbol Device:R
- removed R17, R21, R60: 130, Resistor_SMD:R_0603_1608Metric, symbol Device:R
- removed U8: MAX11125, max1112x-tqfn28:MAX1112x-TQFN-28-1EP_5x5mm_Pitch0.5mm, symbol max1112x:MAX1112x
Connections:
- no-connect marks 4 -> 0
Other:
- note removed: "ADC SPI connected to BANK3 of "ram" sheet"
- note removed: "Audio connected to BANK7 on "gpio" sheet"
- note removed: "JACK pinout for SJ-43516-SMT-TR http://www.cui.com/product/resource/sj-4351x-smt-series.pdf pin 1 - sleeve (GND) pin 2 - tip (left channel) pin 3 - ring1 (right channel) pin 4 - ring2 (video) pin 5 - tip switch pin 6 - ring1 switch"
- note removed: "Output resistance: 75 ohm Internal resistance of FPGA pin: 10 ohm 1/(1/(130+10)+1/(270+10)+1/(549+10)+1/(1100+10))=74.6"
