File: wifi.kicad_sch (KiCad schematic)
At the start: 6 parts, among them U9 ESP32-S3-WROOM-1

Commit message: done with routing
Connections:
- net GN12 renamed GN27
- net GN13 renamed GN26
- net GP12 renamed GP27
- net GP13 renamed GP26
- net WIFI_GPIO15_XTAL_D+ renamed WIFI_XTAL_32K_P
- net WIFI_GPIO16_XTAL_D- renamed WIFI_XTAL_32K_N
Changed lines of the file:
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@@
 		(column_widths 26.67 26.67)
 		(row_heights 3.81 3.81 3.81 3.81 3.81 3.81 3.81 3.81 3.81 3.81 3.81 3.81
-			3.81 3.81 3.81 3.81 3.81
+			3.81 3.81 3.81 3.81 3.81 3.81
 		)
 		(cells
@@
 				)
 			)
-			(table_cell "gn13"
+			(table_cell "gpio_10"
 				(exclude_from_sim no)
 				(at 80.01 128.27 0)
@@
 				)
 			)
+			(table_cell "GPIO_11"
+				(exclude_from_sim no)
+				(at 53.34 132.08 0)
+				(size 26.67 3.81)
+				(margins 0.9525 0.9525 0.9525 0.9525)
+				(span 1 1)
+				(fill
+					(type none)
+				)
+				(effects
+					(font
+						(size 1.524 1.524)
+					)
+					(justify left top)
+				)
+			)
+			(table_cell "gn26"
+				(exclude_from_sim no)
+				(at 80.01 132.08 0)
+				(size 26.67 3.81)
+				(margins 0.9525 0.9525 0.9525 0.9525)
+				(span 1 1)
+				(fill
+					(type none)
+				)
+				(effects
+					(font
+						(size 1.524 1.524)
+					)
+					(justify left top)
+				)
+			)
 			(table_cell "GPIO_12"
 				(exclude_from_sim no)
-				(at 53.34 132.08 0)
-				(size 26.67 3.81)
-				(margins 0.9525 0.9525 0.9525 0.9525)
-				(span 1 1)
-				(fill
-					(type none)
-				)
-				(effects
-					(font
-						(size 1.524 1.524)
-					)
-					(justify left top)
-				)
-			)
-			(table_cell "gp13"
-				(exclude_from_sim no)
-				(at 80.01 132.08 0)
+				(at 53.34 135.89 0)
+				(size 26.67 3.81)
+				(margins 0.9525 0.9525 0.9525 0.9525)
+				(span 1 1)
+				(fill
+					(type none)
+				)
+				(effects
+					(font
+						(size 1.524 1.524)
+					)
+					(justify left top)
+				)
+			)
+			(table_cell "gp26"
+				(exclude_from_sim no)
+				(at 80.01 135.89 0)
 				(size 26.67 3.81)
 				(margins 0.9525 0.9525 0.9525 0.9525)
@@
 			(table_cell "GPIO_13"
 				(exclude_from_sim no)
-				(at 53.34 135.89 0)
-				(size 26.67 3.81)
-				(margins 0.9525 0.9525 0.9525 0.9525)
-				(span 1 1)
-				(fill
-					(type none)
-				)
-				(effects
-					(font
-						(size 1.524 1.524)
-					)
-					(justify left top)
-				)
-			)
-			(table_cell "gn12"
-				(exclude_from_sim no)
-				(at 80.01 135.89 0)
+				(at 53.34 139.7 0)
+				(size 26.67 3.81)
+				(margins 0.9525 0.9525 0.9525 0.9525)
+				(span 1 1)
+				(fill
+					(type none)
+				)
+				(effects
+					(font
+						(size 1.524 1.524)
+					)
+					(justify left top)
+				)
+			)
+			(table_cell "gn27"
+				(exclude_from_sim no)
+				(at 80.01 139.7 0)
 				(size 26.67 3.81)
 				(margins 0.9525 0.9525 0.9525 0.9525)
@@
 			(table_cell "GPIO_14"
 				(exclude_from_sim no)
-				(at 53.34 139.7 0)
-				(size 26.67 3.81)
-				(margins 0.9525 0.9525 0.9525 0.9525)
-				(span 1 1)
-				(fill
-					(type none)
-				)
-				(effects
-					(font
-						(size 1.524 1.524)
-					)
-					(justify left top)
-				)
-			)
-			(table_cell "gp12"
-				(exclude_from_sim no)
-				(at 80.01 139.7 0)
+				(at 53.34 143.51 0)
+				(size 26.67 3.81)
+				(margins 0.9525 0.9525 0.9525 0.9525)
+				(span 1 1)
+				(fill
+					(type none)
+				)
+				(effects
+					(font
+						(size 1.524 1.524)
+					)
+					(justify left top)
+				)
+			)
+			(table_cell "gp27"
+				(exclude_from_sim no)
+				(at 80.01 143.51 0)
 				(size 26.67 3.81)
 				(margins 0.9525 0.9525 0.9525 0.9525)
@@
 			(table_cell "GPIO_38 *done"
 				(exclude_from_sim no)
-				(at 53.34 143.51 0)
+				(at 53.34 147.32 0)
 				(size 26.67 3.81)
 				(margins 0.9525 0.9525 0.9525 0.9525)
@@
 			(table_cell "gpio35"
 				(exclude_from_sim no)
-				(at 80.01 143.51 0)
+				(at 80.01 147.32 0)
 				(size 26.67 3.81)
 				(margins 0.9525 0.9525 0.9525 0.9525)
@@
 			(table_cell "GPIO_46 *done"
 				(exclude_from_sim no)
-				(at 53.34 147.32 0)
+				(at 53.34 151.13 0)
 				(size 26.67 3.81)
 				(margins 0.9525 0.9525 0.9525 0.9525)
@@
 			(table_cell "gpio27"
 				(exclude_from_sim no)
-				(at 80.01 147.32 0)
+				(at 80.01 151.13 0)
 				(size 26.67 3.81)
 				(margins 0.9525 0.9525 0.9525 0.9525)
@@
 			(table_cell "WIFI_USB_D+"
 				(exclude_from_sim no)
-				(at 53.34 151.13 0)
+				(at 53.34 154.94 0)
 				(size 26.67 3.81)
 				(margins 0.9525 0.9525 0.9525 0.9525)
@@
 			(table_cell "P1"
 				(exclude_from_sim no)
-				(at 80.01 151.13 0)
+				(at 80.01 154.94 0)
 				(size 26.67 3.81)
 				(margins 0.9525 0.9525 0.9525 0.9525)
@@
 			(table_cell "WIFI_USB_D-"
 				(exclude_from_sim no)
-				(at 53.34 154.94 0)
+				(at 53.34 158.75 0)
 				(size 26.67 3.81)
 				(margins 0.9525 0.9525 0.9525 0.9525)
@@
 			(table_cell "P2"
 				(exclude_from_sim no)
-				(at 80.01 154.94 0)
+				(at 80.01 158.75 0)
 				(size 26.67 3.81)
 				(margins 0.9525 0.9525 0.9525 0.9525)
@@
 		)
 	)
-	(global_label "GP13"
+	(global_label "GP26"
 		(shape input)
 		(at 238.76 109.22 0)
@@
 		)
 	)
-	(global_label "WIFI_GPIO16_XTAL_D-"
+	(global_label "WIFI_XTAL_32K_N"
 		(shape input)
 		(at 147.32 73.66 180)
@@
 		)
 	)
-	(global_label "GN13"
+	(global_label "GN26"
 		(shape input)
 		(at 238.76 106.68 0)
@@
 		)
 	)
-	(global_label "GP12"
+	(global_label "GP27"
 		(shape input)
 		(at 238.76 114.3 0)
@@
 		)
 	)
-	(global_label "WIFI_GPIO15_XTAL_D+"
+	(global_label "WIFI_XTAL_32K_P"
 		(shape input)
 		(at 147.32 71.12 180)
@@
 		)
 	)
-	(global_label "GN12"
+	(global_label "GN27"
 		(shape input)
 		(at 238.76 111.76 0)

Commit message: fix diff pairs
Connections:
- net WIFI_XTAL_32K_N renamed WIFI_GPIO16
- net WIFI_XTAL_32K_P renamed WIFI_GPIO15
Changed lines of the file:
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@@
 		)
 	)
-	(global_label "WIFI_XTAL_32K_N"
+	(global_label "WIFI_GPIO16"
 		(shape input)
 		(at 147.32 73.66 180)
@@
 		)
 	)
-	(global_label "WIFI_XTAL_32K_P"
+	(global_label "WIFI_GPIO15"
 		(shape input)
 		(at 147.32 71.12 180)
