File: wifi.kicad_sch (KiCad schematic)
At the start: 6 parts, among them U9 ESP32-S3-WROOM-1

Commit message: make MPN reflect mouser part numbers
Parts:
- R38, R56: MPN RC0603FR-0715KL -> 603-RC0603FR-0715KL
- R39: MPN 13-AC0603FR-07549RLCT-ND -> 603-AC0603FR-07549RL
Changed lines of the file:
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@@
 			)
 		)
-		(property "MPN" "RC0603FR-0715KL"
+		(property "MPN" "603-RC0603FR-0715KL"
 			(at 130.81 17.78 90)
 			(hide yes)
@@
 			)
 		)
-		(property "MPN" "RC0603FR-0715KL"
+		(property "MPN" "603-RC0603FR-0715KL"
 			(at 142.24 48.26 90)
 			(hide yes)
@@
 			)
 		)
-		(property "MPN" "13-AC0603FR-07549RLCT-ND"
+		(property "MPN" "603-AC0603FR-07549RL"
 			(at 142.24 58.42 90)
 			(hide yes)
