File: blinkey.kicad_sch (KiCad schematic)
At the start: 10 parts

Commit message: make MPN reflect mouser part numbers
Parts:
- D0, D19: MPN LTST-C170KRKT -> 859-LTST-C170KRKT
- D1: MPN LTST-C170KFKT -> 859-LTST-C170KFKT
- D18: MPN LTST-C170TGKT -> 859-LTST-C170TGKT
- D22: MPN LTST-C170TBKT -> 859-LTST-C170TBKT
- R36, R37, R41, R42, R62: MPN 13-AC0603FR-07549RLCT-ND -> 603-AC0603FR-07549RL
Changed lines of the file:
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@@
 			)
 		)
-		(property "MPN" "13-AC0603FR-07549RLCT-ND"
+		(property "MPN" "603-AC0603FR-07549RL"
 			(at 115.57 116.84 90)
 			(hide yes)
@@
 			)
 		)
-		(property "MPN" "LTST-C170KRKT"
+		(property "MPN" "859-LTST-C170KRKT"
 			(at 115.57 135.89 0)
 			(hide yes)
@@
 			)
 		)
-		(property "MPN" "13-AC0603FR-07549RLCT-ND"
+		(property "MPN" "603-AC0603FR-07549RL"
 			(at 139.7 135.89 90)
 			(hide yes)
@@
 			)
 		)
-		(property "MPN" "13-AC0603FR-07549RLCT-ND"
+		(property "MPN" "603-AC0603FR-07549RL"
 			(at 133.35 64.77 90)
 			(hide yes)
@@
 			)
 		)
-		(property "MPN" "13-AC0603FR-07549RLCT-ND"
+		(property "MPN" "603-AC0603FR-07549RL"
 			(at 133.35 69.85 90)
 			(hide yes)
@@
 			)
 		)
-		(property "MPN" "13-AC0603FR-07549RLCT-ND"
+		(property "MPN" "603-AC0603FR-07549RL"
 			(at 115.57 148.59 90)
 			(hide yes)
@@
 			)
 		)
-		(property "MPN" "LTST-C170KRKT"
+		(property "MPN" "859-LTST-C170KRKT"
 			(at 115.57 64.77 0)
 			(hide yes)
@@
 			)
 		)
-		(property "MPN" "LTST-C170KFKT"
+		(property "MPN" "859-LTST-C170KFKT"
 			(at 115.57 69.85 0)
 			(hide yes)
@@
 			)
 		)
-		(property "MPN" "LTST-C170TBKT"
+		(property "MPN" "859-LTST-C170TBKT"
 			(at 139.7 148.59 0)
 			(hide yes)
@@
 			)
 		)
-		(property "MPN" "LTST-C170TGKT "
+		(property "MPN" "859-LTST-C170TGKT"
 			(at 139.7 116.84 0)
 			(hide yes)
