File: power.kicad_sch (KiCad schematic)
At the start: 41 parts, among them U1 LFE5U-85F-6BG381C, U11 MPM54304GMN-0001

Commit message: update parts for 22uf/1uf. Update footprint for RP* items
Parts:
- C13, C14, C15, C18, C36, C37, C39, C40: Digikey 1276-2413-1-ND -> 311-1900-1-ND; LCSC C29277 -> (none); MPN CC0805ZKY5V5BB226 -> 603-CC805MKX5R6BB226; MPN2 (none) -> CC0805ZKY5V5BB226
- C38: Digikey (none) -> 311-3423-1-ND; MPN (none) -> 603-CC805KRX5R6BB105
- RP4, RP5, RP6: footprint jumper:R_0805_2012Metric_Pad1.29x1.40mm_HandSolder_Jumper_NC -> Resistor_SMD:R_0805_2012Metric_Pad1.20x1.40mm_HandSolder; Digikey (none) -> 311-0.0ARCT-ND; MPN (none) -> 603-RC0805JR-070RL
- U11: Digikey (none) -> 1589-MPM54304GMN-0001-ND

Commit message: interim esp32 change
Parts:
- D27: symbol Device:LED_ALT -> Device:LED
Changed lines of the file:
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@@
 	)
 	(junction
+		(at 191.77 99.06)
+		(diameter 0)
+		(color 0 0 0 0)
+	)
+	(junction
 		(at 219.71 66.04)
 		(diameter 0)
@@
 	)
 	(junction
-		(at 177.8 99.06)
-		(diameter 0)
-		(color 0 0 0 0)
-	)
-	(junction
 		(at 100.33 66.04)
 		(diameter 0)
@@
 	)
 	(junction
-		(at 191.77 99.06)
-		(diameter 0)
-		(color 0 0 0 0)
-	)
-	(junction
 		(at 168.91 66.04)
 		(diameter 0)
@@
 	)
 	(junction
+		(at 177.8 99.06)
+		(diameter 0)
+		(color 0 0 0 0)
+	)
+	(junction
 		(at 184.15 26.67)
 		(diameter 0)
@@
 	(wire
 		(pts
-			(xy 186.632 99.06) (xy 191.77 99.06)
+			(xy 186.69 99.06) (xy 191.77 99.06)
 		)
 		(stroke
@@
 	(wire
 		(pts
-			(xy 177.8 99.06) (xy 181.552 99.06)
+			(xy 177.8 99.06) (xy 181.61 99.06)
 		)
 		(stroke
@@
 	)
 	(symbol
-		(lib_id "Device:LED_ALT")
+		(lib_id "Device:LED")
 		(at 80.01 109.22 90)
 		(unit 1)
@@
 			)
 		)
-		(property "Description" ""
+		(property "Description" "Light emitting diode"
 			(at 80.01 109.22 0)
+			(hide yes)
 			(show_name no)
 			(do_not_autoplace no)
@@
 			)
 		)
+		(property "Sim.Pins" "1=K 2=A"
+			(at 80.01 109.22 0)
+			(hide yes)
+			(show_name no)
+			(do_not_autoplace no)
+			(effects
+				(font
+					(size 1.27 1.27)
+				)
+			)
+		)
 		(pin "1"
 		)
@@
 	(symbol
 		(lib_id "Device:Jumper_NC_Small")
-		(at 184.092 99.06 0)
+		(at 184.15 99.06 0)
 		(unit 1)
 		(body_style 1)
@@
 		(dnp yes)
 		(property "Reference" "RP4"
-			(at 184.092 97.028 0)
+			(at 184.15 97.028 0)
 			(show_name no)
 			(do_not_autoplace no)
@@
 		)
 		(property "Value" "0"
-			(at 184.092 100.33 0)
+			(at 184.15 100.33 0)
 			(show_name no)
 			(do_not_autoplace no)
@@
 		)
 		(property "Footprint" "Resistor_SMD:R_0805_2012Metric_Pad1.20x1.40mm_HandSolder"
-			(at 184.092 99.06 0)
+			(at 184.15 99.06 0)
 			(hide yes)
 			(show_name no)
@@
 		)
 		(property "Datasheet" ""
-			(at 184.092 99.06 0)
+			(at 184.15 99.06 0)
 			(hide yes)
 			(show_name no)
@@
 		)
 		(property "Description" ""
-			(at 184.092 99.06 0)
+			(at 184.15 99.06 0)
 			(show_name no)
 			(do_not_autoplace no)
@@
 		)
 		(property "Mouser_URL" "www.mouser.com"
-			(at 184.092 99.06 0)
+			(at 184.15 99.06 0)
 			(hide yes)
 			(show_name no)
@@
 		)
 		(property "MNF1_URL" "www.yageo.com"
-			(at 184.092 99.06 0)
+			(at 184.15 99.06 0)
 			(hide yes)
 			(show_name no)
@@
 		)
 		(property "EMPTY_MPN" "RC0805JR-070RL"
-			(at 184.092 99.06 0)
+			(at 184.15 99.06 0)
 			(hide yes)
 			(show_name no)
@@
 		)
 		(property "Mouse_r1" "71-RCG08050000Z0EA"
-			(at 184.092 99.06 0)
+			(at 184.15 99.06 0)
 			(hide yes)
 			(show_name no)
@@
 		)
 		(property "Mouse_r2" "603-RC0805JR-070RL"
-			(at 184.092 99.06 0)
+			(at 184.15 99.06 0)
 			(hide yes)
 			(show_name no)
@@
 		)
 		(property "Mouse_r3" "652-CR0805-J/-000ELF"
-			(at 184.092 99.06 0)
+			(at 184.15 99.06 0)
 			(hide yes)
 			(show_name no)
@@
 		)
 		(property "Digike_y1" "YAG1327CT-ND"
-			(at 184.092 99.06 0)
+			(at 184.15 99.06 0)
 			(hide yes)
 			(show_name no)
@@
 		)
 		(property "Note" ""
-			(at 184.092 99.06 0)
+			(at 184.15 99.06 0)
 			(hide yes)
 			(show_name no)
@@
 		)
 		(property "MPN" "603-RC0805JR-070RL"
-			(at 184.092 99.06 0)
+			(at 184.15 99.06 0)
 			(hide yes)
 			(show_name no)
@@
 		)
 		(property "Arrow" ""
-			(at 184.092 99.06 0)
+			(at 184.15 99.06 0)
 			(hide yes)
 			(show_name no)
@@
 		)
 		(property "DatasheetLC" ""
-			(at 184.092 99.06 0)
+			(at 184.15 99.06 0)
 			(hide yes)
 			(show_name no)
@@
 		)
 		(property "LCS_C2" ""
-			(at 184.092 99.06 0)
+			(at 184.15 99.06 0)
 			(hide yes)
 			(show_name no)
@@
 		)
 		(property "MP_N4" ""
-			(at 184.092 99.06 0)
+			(at 184.15 99.06 0)
 			(hide yes)
 			(show_name no)
@@
 		)
 		(property "MP_N5" ""
-			(at 184.092 99.06 0)
+			(at 184.15 99.06 0)
 			(hide yes)
 			(show_name no)
@@
 		)
 		(property "Vertical" ""
-			(at 184.092 99.06 0)
+			(at 184.15 99.06 0)
 			(hide yes)
 			(show_name no)
@@
 		)
 		(property "price100_Mouser" ""
-			(at 184.092 99.06 0)
+			(at 184.15 99.06 0)
 			(hide yes)
 			(show_name no)
@@
 		)
 		(property "price1200_Chip1stop" ""
-			(at 184.092 99.06 0)
+			(at 184.15 99.06 0)
 			(hide yes)
 			(show_name no)
@@
 		)
 		(property "price300_LCSC" ""
-			(at 184.092 99.06 0)
+			(at 184.15 99.06 0)
 			(hide yes)
 			(show_name no)
@@
 		)
 		(property "price300_Vertical" ""
-			(at 184.092 99.06 0)
+			(at 184.15 99.06 0)
 			(hide yes)
 			(show_name no)
@@
 		)
 		(property "price_Arrow" ""
-			(at 184.092 99.06 0)
+			(at 184.15 99.06 0)
 			(hide yes)
 			(show_name no)
@@
 		)
 		(property "Digikey" "311-0.0ARCT-ND"
-			(at 184.092 99.06 0)
+			(at 184.15 99.06 0)
 			(hide yes)
 			(show_name no)

Commit message: switch to smaller pts810 button
Parts:
- B0: value PTS645 -> PTS810SJM250SMTR LFS; footprint Button_Switch_SMD:SW_SPST_PTS645 -> pts810:PTS810_CNK; Digikey CKN9088CT-ND -> CKN10502CT-ND; Koncar FSW001 -> (none); LCSC C285463 -> C116501; MNF1_URL www.ckswitches.com -> (none); MPN PTS645SL50SMTR92 LFS -> 611-PTS810SJM250SMTR; Mouser 611-PTS645SL50SMTR92 -> (none); Newar_k2 79AH5908 -> (none); Newark 15N4500 -> 26AH0019; price700_LCSC 0.09966$ -> (none)
Changed lines of the file:
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@@
 			)
 		)
-		(property "Value" "PTS645"
-			(at 22.86 64.77 0)
+		(property "Value" "PTS810SJM250SMTR LFS"
+			(at 27.94 62.23 0)
 			(show_name no)
 			(do_not_autoplace no)
@@
 			)
 		)
-		(property "Footprint" "Button_Switch_SMD:SW_SPST_PTS645"
+		(property "Footprint" "pts810:PTS810_CNK"
 			(at 26.67 97.79 0)
 			(hide yes)
@@
 			)
 		)
-		(property "Datasheet" "http://www.ckswitches.com/media/1471/pts645.pdf"
+		(property "Datasheet" "https://www.littelfuse.com/assetdocs/littelfuse-c-k-tactile-pts810-series-datasheet?assetguid=f1e4bc97-66e9-4beb-99c6-eaef0bd3bff4"
 			(at 26.67 97.79 0)
 			(hide yes)
@@
 			)
 		)
-		(property "Description" ""
-			(at 26.67 67.31 0)
+		(property "Description" "SWITCH TACTILE SPST-NO 0.05A 16V"
+			(at 26.416 62.23 0)
+			(hide yes)
 			(show_name no)
 			(do_not_autoplace no)
@@
 			)
 		)
-		(property "MNF1_URL" "www.ckswitches.com"
+		(property "MPN" "611-PTS810SJM250SMTR"
 			(at 26.67 67.31 0)
 			(hide yes)
@@
 			)
 		)
-		(property "MPN" "PTS645SL50SMTR92 LFS"
-			(at 26.67 67.31 0)
-			(hide yes)
-			(show_name no)
-			(do_not_autoplace no)
-			(effects
-				(font
-					(size 1.524 1.524)
-				)
-			)
-		)
-		(property "Mouser" "611-PTS645SL50SMTR92"
+		(property "Digikey" "CKN10502CT-ND"
 			(at 26.67 67.31 0)
 			(hide yes)
@@
 			)
 		)
-		(property "Digikey" "CKN9088CT-ND"
+		(property "Newark" "26AH0019"
 			(at 26.67 67.31 0)
 			(hide yes)
@@
 			)
 		)
-		(property "Newark" "15N4500"
-			(at 26.67 67.31 0)
-			(hide yes)
-			(show_name no)
-			(do_not_autoplace no)
-			(effects
-				(font
-					(size 1.27 1.27)
-				)
-			)
-		)
-		(property "Newar_k2" "79AH5908"
-			(at 26.67 67.31 0)
-			(hide yes)
-			(show_name no)
-			(do_not_autoplace no)
-			(effects
-				(font
-					(size 1.27 1.27)
-				)
-			)
-		)
-		(property "LCSC" "C285463"
-			(at 26.67 67.31 0)
-			(hide yes)
-			(show_name no)
-			(do_not_autoplace no)
-			(effects
-				(font
-					(size 1.27 1.27)
-				)
-			)
-		)
-		(property "price700_LCSC" "0.09966$"
-			(at 26.67 67.31 0)
-			(hide yes)
-			(show_name no)
-			(do_not_autoplace no)
-			(effects
-				(font
-					(size 1.27 1.27)
-				)
-			)
-		)
-		(property "Koncar" "FSW001"
+		(property "LCSC" "C116501"
 			(at 26.67 67.31 0)
 			(hide yes)
@@
 				)
 			)
-		)
-		(property "Arrow" ""
-			(at 26.67 67.31 0)
-			(hide yes)
-			(show_name no)
-			(do_not_autoplace no)
-			(effects
-				(font
-					(size 1.524 1.524)
-				)
-			)
-		)
-		(property "DatasheetLC" ""
-			(at 26.67 67.31 0)
-			(hide yes)
-			(show_name no)
-			(do_not_autoplace no)
-			(effects
-				(font
-					(size 1.524 1.524)
-				)
-			)
-		)
-		(property "LCS_C2" ""
-			(at 26.67 67.31 0)
-			(hide yes)
-			(show_name no)
-			(do_not_autoplace no)
-			(effects
-				(font
-					(size 1.524 1.524)
-				)
-			)
-		)
-		(property "MP_N4" ""
-			(at 26.67 67.31 0)
-			(hide yes)
-			(show_name no)
-			(do_not_autoplace no)
-			(effects
-				(font
-					(size 1.524 1.524)
-				)
-			)
-		)
-		(property "MP_N5" ""
-			(at 26.67 67.31 0)
-			(hide yes)
-			(show_name no)
-			(do_not_autoplace no)
-			(effects
-				(font
-					(size 1.524 1.524)
-				)
-			)
-		)
-		(property "Vertical" ""
-			(at 26.67 67.31 0)
-			(hide yes)
-			(show_name no)
-			(do_not_autoplace no)
-			(effects
-				(font
-					(size 1.524 1.524)
-				)
-			)
-		)
-		(property "price100_Mouser" ""
-			(at 26.67 67.31 0)
-			(hide yes)
-			(show_name no)
-			(do_not_autoplace no)
-			(effects
-				(font
-					(size 1.524 1.524)
-				)
-			)
-		)
-		(property "price1200_Chip1stop" ""
-			(at 26.67 67.31 0)
-			(hide yes)
-			(show_name no)
-			(do_not_autoplace no)
-			(effects
-				(font
-					(size 1.524 1.524)
-				)
-			)
-		)
-		(property "price300_LCSC" ""
-			(at 26.67 67.31 0)
-			(hide yes)
-			(show_name no)
-			(do_not_autoplace no)
-			(effects
-				(font
-					(size 1.524 1.524)
-				)
-			)
-		)
-		(property "price300_Vertical" ""
-			(at 26.67 67.31 0)
-			(hide yes)
-			(show_name no)
-			(do_not_autoplace no)
-			(effects
-				(font
-					(size 1.524 1.524)
-				)
-			)
-		)
-		(property "price_Arrow" ""
-			(at 26.67 67.31 0)
-			(hide yes)
-			(show_name no)
-			(do_not_autoplace no)
-			(effects
-				(font
-					(size 1.524 1.524)
-				)
-			)

Commit message: done with routing
Parts:
- C48, C49, C50, C51: now not fitted; now left out of the parts list
Changed lines of the file:
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@@
 		(body_style 1)
 		(exclude_from_sim no)
-		(in_bom yes)
-		(on_board yes)
+		(in_bom no)
+		(on_board no)
 		(in_pos_files yes)
-		(dnp no)
+		(dnp yes)
 		(property "Reference" "C50"
 			(at 40.005 90.17 0)
@@
 		(body_style 1)
 		(exclude_from_sim no)
-		(in_bom yes)
-		(on_board yes)
+		(in_bom no)
+		(on_board no)
 		(in_pos_files yes)
-		(dnp no)
+		(dnp yes)
 		(property "Reference" "#PWR036"
 			(at 39.37 102.87 0)
@@
 		(body_style 1)
 		(exclude_from_sim no)
-		(in_bom yes)
-		(on_board yes)
+		(in_bom no)
+		(on_board no)
 		(in_pos_files yes)
-		(dnp no)
+		(dnp yes)
 		(property "Reference" "#PWR035"
 			(at 39.37 92.71 0)
@@
 		(body_style 1)
 		(exclude_from_sim no)
-		(in_bom yes)
-		(on_board yes)
+		(in_bom no)
+		(on_board no)
 		(in_pos_files yes)
-		(dnp no)
+		(dnp yes)
 		(property "Reference" "#PWR031"
 			(at 26.67 102.87 0)
@@
 		(body_style 1)
 		(exclude_from_sim no)
-		(in_bom yes)
-		(on_board yes)
+		(in_bom no)
+		(on_board no)
 		(in_pos_files yes)
-		(dnp no)
+		(dnp yes)
 		(property "Reference" "C48"
 			(at 27.305 90.17 0)
@@
 		(body_style 1)
 		(exclude_from_sim no)
-		(in_bom yes)
-		(on_board yes)
+		(in_bom no)
+		(on_board no)
 		(in_pos_files yes)
-		(dnp no)
+		(dnp yes)
 		(property "Reference" "#PWR037"
 			(at 45.72 92.71 0)
@@
 		(body_style 1)
 		(exclude_from_sim no)
-		(in_bom yes)
-		(on_board yes)
+		(in_bom no)
+		(on_board no)
 		(in_pos_files yes)
-		(dnp no)
+		(dnp yes)
 		(property "Reference" "#PWR038"
 			(at 45.72 102.87 0)
@@
 		(body_style 1)
 		(exclude_from_sim no)
-		(in_bom yes)
-		(on_board yes)
+		(in_bom no)
+		(on_board no)
 		(in_pos_files yes)
-		(dnp no)
+		(dnp yes)
 		(property "Reference" "C51"
 			(at 46.355 90.17 0)
@@
 		(body_style 1)
 		(exclude_from_sim no)
-		(in_bom yes)
-		(on_board yes)
+		(in_bom no)
+		(on_board no)
 		(in_pos_files yes)
-		(dnp no)
+		(dnp yes)
 		(property "Reference" "#PWR034"
 			(at 33.02 102.87 0)
@@
 		(body_style 1)
 		(exclude_from_sim no)
-		(in_bom yes)
-		(on_board yes)
+		(in_bom no)
+		(on_board no)
 		(in_pos_files yes)
-		(dnp no)
+		(dnp yes)
 		(property "Reference" "C49"
 			(at 33.655 90.17 0)
@@
 		(body_style 1)
 		(exclude_from_sim no)
-		(in_bom yes)
-		(on_board yes)
+		(in_bom no)
+		(on_board no)
 		(in_pos_files yes)
-		(dnp no)
+		(dnp yes)
 		(property "Reference" "#PWR087"
 			(at 33.02 92.71 0)
@@
 		(body_style 1)
 		(exclude_from_sim no)
-		(in_bom yes)
-		(on_board yes)
+		(in_bom no)
+		(on_board no)
 		(in_pos_files yes)
-		(dnp no)
+		(dnp yes)
 		(property "Reference" "#PWR086"
 			(at 26.67 92.71 0)

Commit message: add i2c header
Parts:
- added J6: I2C Header, Connector_PinHeader_2.54mm:PinHeader_1x02_P2.54mm_Vertical, symbol Connector:Conn_01x02_Socket
Connections:
- net I2C_SCL: now also J6.2 (Pin_2)
- net I2C_SDA: now also J6.1 (Pin_1)
- no-connect marks 7 -> 5
Changed lines of the file:
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@@
 	)
 	(no_connect
-		(at 104.14 139.7)
-	)
-	(no_connect
 		(at 144.78 162.56)
 	)
@@
 	)
 	(no_connect
-		(at 104.14 142.24)
-	)
-	(no_connect
 		(at 144.78 154.94)
 	)
@@
 	(wire
 		(pts
+			(xy 92.71 139.7) (xy 104.14 139.7)
+		)
+		(stroke
+			(width 0)
+			(type default)
+		)
+	)
+	(wire
+		(pts
 			(xy 129.54 20.32) (xy 129.54 26.67)
 		)
@@
 	(wire
 		(pts
+			(xy 92.71 142.24) (xy 104.14 142.24)
+		)
+		(stroke
+			(width 0)
+			(type default)
+		)
+	)
+	(wire
+		(pts
 			(xy 111.76 26.67) (xy 111.76 29.21)
 		)
@@
 		)
 	)
-	(label "I2C_SCL"
-		(at 104.14 142.24 180)
-		(effects
-			(font
-				(size 1.524 1.524)
-			)
-			(justify right bottom)
-		)
-	)
 	(label "LED_PWRBAD"
 		(at 80.01 121.92 180)
@@
 		)
 	)
-	(label "I2C_SDA"
-		(at 104.14 139.7 180)
+	(label "P3V3"
+		(at 154.94 99.06 0)
 		(effects
 			(font
 				(size 1.524 1.524)
 			)
-			(justify right bottom)
+			(justify left bottom)
 		)
 	)
-	(label "P3V3"
-		(at 154.94 99.06 0)
+	(global_label "I2C_SCL"
+		(shape input)
+		(at 96.52 142.24 270)
 		(effects
 			(font
 				(size 1.524 1.524)
 			)
-			(justify left bottom)
+			(justify right)
+		)
+		(property "Intersheetrefs" "${INTERSHEET_REFS}"
+			(at 96.52 142.24 90)
+			(hide yes)
+			(show_name no)
+			(do_not_autoplace no)
+			(effects
+				(font
+					(size 1.27 1.27)
+				)
+			)
 		)
 	)
@@
 		)
 	)
+	(global_label "I2C_SDA"
+		(shape input)
+		(at 96.52 139.7 90)
+		(effects
+			(font
+				(size 1.524 1.524)
+			)
+			(justify left)
+		)
+		(property "Intersheetrefs" "${INTERSHEET_REFS}"
+			(at 96.52 139.7 90)
+			(hide yes)
+			(show_name no)
+			(do_not_autoplace no)
+			(effects
+				(font
+					(size 1.27 1.27)
+				)
+			)
+		)
+	)
 	(symbol
 		(lib_id "power:GND")
@@
 					(unit 1)
 				)
+			)
+		)
+	)
+	(symbol
+		(lib_id "Connector:Conn_01x02_Socket")
+		(at 87.63 139.7 0)
+		(mirror y)
+		(unit 1)
+		(body_style 1)
+		(exclude_from_sim no)
+		(in_bom yes)
+		(on_board yes)
+		(in_pos_files yes)
+		(dnp no)
+		(property "Reference" "J6"
+			(at 86.36 139.6999 0)
+			(show_name no)
+			(do_not_autoplace no)
+			(effects
+				(font
+					(size 1.27 1.27)
+				)
+				(justify left)
+			)
+		)
+		(property "Value" "I2C Header"
+			(at 90.932 145.034 0)
+			(show_name no)
+			(do_not_autoplace no)
+			(effects
+				(font
+					(size 1.27 1.27)
+				)
+				(justify left)
+			)
+		)
+		(property "Footprint" "Connector_PinHeader_2.54mm:PinHeader_1x02_P2.54mm_Vertical"
+			(at 87.63 139.7 0)
+			(hide yes)
+			(show_name no)
+			(do_not_autoplace no)
+			(effects
+				(font
+					(size 1.27 1.27)
+				)
+			)
+		)
+		(property "Datasheet" ""
+			(at 87.63 139.7 0)
+			(hide yes)
+			(show_name no)
+			(do_not_autoplace no)
+			(effects
+				(font
+					(size 1.27 1.27)
+				)
+			)
+		)
+		(property "Description" "Generic connector, single row, 01x02, script generated"
+			(at 87.63 139.7 0)
+			(hide yes)
+			(show_name no)
+			(do_not_autoplace no)
+			(effects
+				(font
+					(size 1.27 1.27)
+				)
+			)
+		)
+		(pin "2"
+		)
+		(pin "1"
+		)
+		(instances
+			(project "ulx3s"
+				(path "/49a43414-f3c1-43b2-ad20-ac3166075f21/00000000-0000-0000-0000-000058d51cad"
+					(reference "J6")
+					(unit 1)
+				)

Commit message: switch to usb-c. upgrade to v1.0.4
Parts:
- J6: now left out of the parts list
Changed lines of the file:
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@@
 		(body_style 1)
 		(exclude_from_sim no)
-		(in_bom yes)
+		(in_bom no)
 		(on_board yes)
 		(in_pos_files yes)

Commit message: make MPN reflect mouser part numbers
Parts:
- C17, C19, C20: MPN CC0805MRX5R6BB225 -> 603-CC805MRX5R6BB225
- C25, C26, C27, C28, C29, C30, C31, C32, C53: MPN CC0603JRX7R8BB223 -> 603-CC603JRX7R8BB223
- C60: MPN CC0603KRX7R8BB224 -> 603-CC603KRX7R8BB224
- D27: MPN LTST-C170KRKT -> 859-LTST-C170KRKT
- R34: MPN 13-AC0603FR-071K1LCT-ND -> 603-AC0603FR-071K1L
- RA4, RA5, RA6: MPN RC0603FR-0715KL -> 603-RC0603FR-0715KL
- RB4: MPN RT0603FRE073K3L -> 603-RT0603FRE073K3L
- RB5: MPN RC0603FR-1018KL -> 603-RC0603FR-1018KL
- U1: MPN LFE5U-85F-6BG381C -> 842-LFE5U85F6BG381C
Changed lines of the file:
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@@
 			)
 		)
-		(property "MPN" "LFE5U-85F-6BG381C"
+		(property "MPN" "842-LFE5U85F6BG381C"
 			(at 157.48 45.72 0)
 			(hide yes)
@@
 			)
 		)
-		(property "MPN" "CC0603JRX7R8BB223"
+		(property "MPN" "603-CC603JRX7R8BB223"
 			(at 21.59 153.67 0)
 			(hide yes)
@@
 			)
 		)
-		(property "MPN" "CC0603JRX7R8BB223"
+		(property "MPN" "603-CC603JRX7R8BB223"
 			(at 41.91 153.67 0)
 			(hide yes)
@@
 			)
 		)
-		(property "MPN" "CC0603JRX7R8BB223"
+		(property "MPN" "603-CC603JRX7R8BB223"
 			(at 27.94 115.57 0)
 			(hide yes)
@@
 			)
 		)
-		(property "MPN" "CC0603JRX7R8BB223"
+		(property "MPN" "603-CC603JRX7R8BB223"
 			(at 34.29 115.57 0)
 			(hide yes)
@@
 			)
 		)
-		(property "MPN" "CC0603JRX7R8BB223"
+		(property "MPN" "603-CC603JRX7R8BB223"
 			(at 27.94 134.62 0)
 			(hide yes)
@@
 			)
 		)
-		(property "MPN" "CC0603JRX7R8BB223"
+		(property "MPN" "603-CC603JRX7R8BB223"
 			(at 34.29 134.62 0)
 			(hide yes)
@@
 			)
 		)
-		(property "MPN" "CC0603JRX7R8BB223"
+		(property "MPN" "603-CC603JRX7R8BB223"
 			(at 34.29 153.67 0)
 			(hide yes)
@@
 			)
 		)
-		(property "MPN" "CC0603JRX7R8BB223"
+		(property "MPN" "603-CC603JRX7R8BB223"
 			(at 27.94 153.67 0)
 			(hide yes)
@@
 			)
 		)
-		(property "MPN" "CC0603JRX7R8BB223"
+		(property "MPN" "603-CC603JRX7R8BB223"
 			(at 48.26 153.67 0)
 			(hide yes)
@@
 			)
 		)
-		(property "MPN" "CC0603KRX7R8BB224"
+		(property "MPN" "603-CC603KRX7R8BB224"
 			(at 26.67 71.12 90)
 			(hide yes)
@@
 			)
 		)
-		(property "MPN" "CC0805MRX5R6BB225"
+		(property "MPN" "603-CC805MRX5R6BB225"
 			(at 46.99 20.32 0)
 			(hide yes)
@@
 			)
 		)
-		(property "MPN" "RC0603FR-0715KL"
+		(property "MPN" "603-RC0603FR-0715KL"
 			(at 154.94 138.43 90)
 			(hide yes)
@@
 			)
 		)
-		(property "MPN" "RC0603FR-0715KL"
+		(property "MPN" "603-RC0603FR-0715KL"
 			(at 154.94 102.87 90)
 			(hide yes)
@@
 			)
 		)
-		(property "MPN" "RT0603FRE073K3L"
+		(property "MPN" "603-RT0603FRE073K3L"
 			(at 154.94 110.49 90)
 			(hide yes)
@@
 			)
 		)
-		(property "MPN" "RC0603FR-0715KL"
+		(property "MPN" "603-RC0603FR-0715KL"
 			(at 154.94 123.19 90)
 			(hide yes)
@@
 			)
 		)
-		(property "MPN" "LTST-C170KRKT"
+		(property "MPN" "859-LTST-C170KRKT"
 			(at 80.01 109.22 0)
 			(hide yes)
@@
 			)
 		)
-		(property "MPN" "13-AC0603FR-071K1LCT-ND"
+		(property "MPN" "603-AC0603FR-071K1L"
 			(at 83.82 121.92 90)
 			(hide yes)
@@
 			)
 		)
-		(property "MPN" "RC0603FR-1018KL"
+		(property "MPN" "603-RC0603FR-1018KL"
 			(at 161.29 127 90)
 			(hide yes)
@@
 			)
 		)
-		(property "MPN" "CC0805MRX5R6BB225"
+		(property "MPN" "603-CC805MRX5R6BB225"
 			(at 125.73 20.32 0)
 			(hide yes)
@@
 			)
 		)
-		(property "MPN" "CC0805MRX5R6BB225"
+		(property "MPN" "603-CC805MRX5R6BB225"
 			(at 102.87 20.32 0)
 			(hide yes)
