File: flash.kicad_sch (KiCad schematic)
At the start: 13 parts, among them U1 LFE5U-85F-6BG381C, U10 IS25LP128F-JBLE

Commit message: make MPN reflect mouser part numbers
Parts:
- D28, D29: MPN 1N4148WS -> 512-1N4148WS
- R11, R12, R27, R28: MPN RC0603FR-0710KL -> 603-RC0603FR-0710KL
- R29: MPN 13-AC0603FR-071K1LCT-ND -> 603-AC0603FR-071K1L
- R31, R32, R33: MPN RC0603FR-0715KL -> 603-RC0603FR-0715KL
- U1: MPN LFE5U-85F-6BG381C -> 842-LFE5U85F6BG381C
- U10: MPN IS25LP128F-JBLE -> 870-IS25LP128F-JBLE
Changed lines of the file:
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@@
 			)
 		)
-		(property "MPN" "IS25LP128F-JBLE"
+		(property "MPN" "870-IS25LP128F-JBLE"
 			(at 92.71 110.49 0)
 			(hide yes)
@@
 			)
 		)
-		(property "MPN" "RC0603FR-0710KL"
+		(property "MPN" "603-RC0603FR-0710KL"
 			(at 87.63 59.69 90)
 			(hide yes)
@@
 			)
 		)
-		(property "MPN" "RC0603FR-0710KL"
+		(property "MPN" "603-RC0603FR-0710KL"
 			(at 92.71 59.69 90)
 			(hide yes)
@@
 			)
 		)
-		(property "MPN" "13-AC0603FR-071K1LCT-ND"
+		(property "MPN" "603-AC0603FR-071K1L"
 			(at 97.79 59.69 90)
 			(hide yes)
@@
 			)
 		)
-		(property "MPN" "RC0603FR-0710KL"
+		(property "MPN" "603-RC0603FR-0710KL"
 			(at 77.47 59.69 90)
 			(hide yes)
@@
 			)
 		)
-		(property "MPN" "RC0603FR-0710KL"
+		(property "MPN" "603-RC0603FR-0710KL"
 			(at 82.55 59.69 90)
 			(hide yes)
@@
 			)
 		)
-		(property "MPN" "RC0603FR-0715KL"
+		(property "MPN" "603-RC0603FR-0715KL"
 			(at 132.08 59.69 90)
 			(hide yes)
@@
 			)
 		)
-		(property "MPN" "RC0603FR-0715KL"
+		(property "MPN" "603-RC0603FR-0715KL"
 			(at 137.16 59.69 90)
 			(hide yes)
@@
 			)
 		)
-		(property "MPN" "RC0603FR-0715KL"
+		(property "MPN" "603-RC0603FR-0715KL"
 			(at 142.24 59.69 90)
 			(hide yes)
@@
 			)
 		)
-		(property "MPN" "LFE5U-85F-6BG381C"
+		(property "MPN" "842-LFE5U85F6BG381C"
 			(at 184.15 114.3 0)
 			(hide yes)
@@
 			)
 		)
-		(property "MPN" "1N4148WS"
+		(property "MPN" "512-1N4148WS"
 			(at 127 90.17 0)
 			(hide yes)
@@
 			)
 		)
-		(property "MPN" "1N4148WS"
+		(property "MPN" "512-1N4148WS"
 			(at 127 86.36 0)
 			(hide yes)
