File: gpdi.kicad_sch (KiCad schematic)
At the start: 21 parts, among them U1 LFE5U-85F-6BG381C, U11 PCA9306D

Commit message: remove unneeded components from schema
Parts:
- removed C18: 100pF, Capacitor_SMD:C_0603_1608Metric, symbol Device:C
- removed C38, C39, C40, C41, C42, C43, C44, C45: 22nF, Capacitor_SMD:C_0603_1608Metric, symbol Device:C
- removed D30: 3.6V, Diode_SMD:D_SOD-323_HandSoldering, symbol Device:D_Zener_Small_ALT
- removed GPDI1: GPDI-D, conn-fci:CONN-10029449-111RLF, symbol hdmi-d:HDMI-D
- removed R22, R23: 3.3k, Resistor_SMD:R_0603_1608Metric, symbol Device:R
- removed R24: 100k, Resistor_SMD:R_0603_1608Metric, symbol Device:R
- removed R25, R26: 4.7k, Resistor_SMD:R_0603_1608Metric, symbol Device:R
- removed R55: 10k, Resistor_SMD:R_0603_1608Metric, symbol Device:R
- removed R61, R67: 549, Resistor_SMD:R_0603_1608Metric, symbol Device:R
- removed U11: PCA9306D, SM8:SM8, symbol pca9306d:PCA9306D
Connections:
- no-connect marks 4 -> 17
Other:
- note removed: "i2c shared with RTC on "power" sheet"
- note removed: "v1.9: VCC1=3.3V EN=5V"

Commit message: start to normalize bom
Parts:
- U1: Digikey (none) -> 220-2177-ND; LCSC (none) -> C446029
Changed lines of the file:
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@@
+			)
+		)
+		(property "LCSC" "C446029"
+			(at 91.44 73.66 0)
+			(effects
+				(font
+					(size 1.27 1.27)
+				)
+				(hide yes)
+			)
+		)
+		(property "Digikey" "220-2177-ND"
+			(at 91.44 73.66 0)
+			(effects
+				(font
+					(size 1.27 1.27)
+				)
+				(hide yes)
 			)
 		)

Commit message: remove US2 port
Connections:
- no-connect marks 17 -> 21
Changed lines of the file:
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@@
+	)
+	(no_connect
+		(at 110.49 71.12)
 	)
 	(no_connect
@@
 	(no_connect
 		(at 72.39 68.58)
+	)
+	(no_connect
+		(at 72.39 91.44)
 	)
 	(no_connect
@@
 	)
 	(no_connect
+		(at 110.49 91.44)
+	)
+	(no_connect
+		(at 72.39 71.12)
+	)
+	(no_connect

Commit message: make MPN reflect mouser part numbers
Parts:
- U1: MPN LFE5U-85F-6BG381C -> 842-LFE5U85F6BG381C
Changed lines of the file:
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@@
 			)
 		)
-		(property "MPN" "LFE5U-85F-6BG381C"
+		(property "MPN" "842-LFE5U85F6BG381C"
 			(at 91.44 73.66 0)
 			(hide yes)

Commit message: update footprints to include additional border. add i2c resistors
Parts:
- U1: Mouser_URL www.mouser.com -> (none)
Changed lines of the file:
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@@
 			)
 		)
-		(property "Datasheet" "http://www.latticesemi.com/~/media/LatticeSemi/Documents/DataSheets/ECP5/FPGA-DS-02012.pdf"
+		(property "Datasheet" "https://www.mouser.com/datasheet/3/248/1/FPGA_DS_02012_3_4_ECP5_ECP5G_Family_Data_Sheet.pdf"
 			(at 64.77 49.53 0)
 			(hide yes)
@@
 			(at 91.44 73.66 0)
 			(hide yes)
-			(show_name no)
-			(do_not_autoplace no)
-			(effects
-				(font
-					(size 1.524 1.524)
-				)
-			)
-		)
-		(property "Mouser_URL" "www.mouser.com"
-			(at 91.44 73.66 0)
-			(hide yes)
