File: serdes.kicad_sch (KiCad schematic)
At the start: 1 part, among them U1 LFE5U-85F-6BG381C

Commit message: make MPN reflect mouser part numbers
Parts:
- U1: MPN LFE5U-85F-6BG381C -> 842-LFE5U85F6BG381C
Changed lines of the file:
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@@
 			)
 		)
-		(property "MPN" "LFE5U-85F-6BG381C"
+		(property "MPN" "842-LFE5U85F6BG381C"
 			(at 144.78 72.39 0)
 			(hide yes)

Commit message: update footprints to include additional border. add i2c resistors
Parts:
- U1: Digike_y2 220-2071-ND -> (none); Koncar FU004 -> (none); LowCost 842-LFE5U12F6BG381C -> (none); MFG1 Lattice -> (none); MFG2 Lattice -> (none); MNF1_URL www.latticesemi.com -> (none); MNF2_URL www.latticesemi.com -> (none); MP_N2 LFE5U-12F-6BG381C -> (none); Mouser 842-LFE5U85F6BG381C -> (none); Side T -> (none); price100_Mouse 22.82$ -> (none)
Changed lines of the file:
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@@
 			)
 		)
-		(property "Datasheet" "http://www.latticesemi.com/~/media/LatticeSemi/Documents/ApplicationNotes/EH/TN1261.pdf?document_id=50463"
+		(property "Datasheet" "https://www.mouser.com/datasheet/3/248/1/FPGA_DS_02012_3_4_ECP5_ECP5G_Family_Data_Sheet.pdf"
 			(at 118.11 48.26 0)
 			(hide yes)
@@
 			)
 		)
-		(property "MFG1" "Lattice"
-			(at 144.78 72.39 0)
-			(hide yes)
-			(show_name no)
-			(do_not_autoplace no)
-			(effects
-				(font
-					(size 1.27 1.27)
-				)
-			)
-		)
-		(property "MNF1_URL" "www.latticesemi.com"
-			(at 144.78 72.39 0)
-			(hide yes)
-			(show_name no)
-			(do_not_autoplace no)
-			(effects
-				(font
-					(size 1.27 1.27)
-				)
-			)
-		)
 		(property "MPN" "842-LFE5U85F6BG381C"
 			(at 144.78 72.39 0)
@@
 				(font
 					(size 1.524 1.524)
-				)
-			)
-		)
-		(property "MFG2" "Lattice"
-			(at 144.78 72.39 0)
-			(hide yes)
-			(show_name no)
-			(do_not_autoplace no)
-			(effects
-				(font
-					(size 1.27 1.27)
-				)
-			)
-		)
-		(property "MNF2_URL" "www.latticesemi.com"
-			(at 144.78 72.39 0)
-			(hide yes)
-			(show_name no)
-			(do_not_autoplace no)
-			(effects
-				(font
-					(size 1.27 1.27)
-				)
-			)
-		)
-		(property "MP_N2" "LFE5U-12F-6BG381C"
-			(at 144.78 72.39 0)
-			(hide yes)
-			(show_name no)
-			(do_not_autoplace no)
-			(effects
-				(font
-					(size 1.27 1.27)
-				)
-			)
-		)
-		(property "Mouser" "842-LFE5U85F6BG381C"
-			(at 144.78 72.39 0)
-			(hide yes)
-			(show_name no)
-			(do_not_autoplace no)
-			(effects
-				(font
-					(size 1.524 1.524)
-				)
-			)
-		)
-		(property "price100_Mouse" "22.82$"
-			(at 144.78 72.39 0)
-			(hide yes)
-			(show_name no)
-			(do_not_autoplace no)
-			(effects
-				(font
-					(size 1.27 1.27)
 				)
 			)
@@
 			)
 		)
-		(property "Digike_y2" "220-2071-ND"
-			(at 144.78 72.39 0)
-			(hide yes)
-			(show_name no)
-			(do_not_autoplace no)
-			(effects
-				(font
-					(size 1.27 1.27)
-				)
-			)
-		)
 		(property "LCSC" "C446029"
 			(at 144.78 72.39 0)
 			(hide yes)
-			(show_name no)
-			(do_not_autoplace no)
-			(effects
-				(font
-					(size 1.27 1.27)
-				)
-			)
-		)
-		(property "LowCost" "842-LFE5U12F6BG381C"
-			(at 144.78 72.39 0)
-			(hide yes)
-			(show_name no)
-			(do_not_autoplace no)
-			(effects
-				(font
-					(size 1.27 1.27)
-				)
-			)
-		)
-		(property "Koncar" "FU004"
-			(at 144.78 72.39 0)
-			(hide yes)
-			(show_name no)
-			(do_not_autoplace no)
-			(effects
-				(font
-					(size 1.27 1.27)
-				)
-			)
-		)
-		(property "Side" "T"
-			(at 144.78 72.39 0)
-			(hide yes)
