File: ulx3s.kicad_sch (KiCad schematic)
At the start: 11 parts

Commit message: add mounting holes. reposition ft231x. use nsleep
Parts:
- H1, H2, H3: value HOLE -> HALFHOLE; footprint Mounting_Holes:MountingHole_3.2mm_M3_ISO14580_Pad -> Mounting_Holes:MountingHole_2.2mm_M2_custom_HALF; symbol Connector_Generic:Conn_01x01 -> Mechanical:MountingHole
- H4: footprint Mounting_Holes:MountingHole_3.2mm_M3_ISO14580_Pad -> Mounting_Holes:MountingHole_2.2mm_M2_custom; symbol Connector_Generic:Conn_01x01 -> Mechanical:MountingHole
Connections:
- removed net GND: H1.1 (Pin_1), H2.1 (Pin_1), H3.1 (Pin_1), H4.1 (Pin_1)
